File: PCIexpress_x1_low/decap.kicad_sch (KiCad schematic)
At the start: 2 parts

Commit message: saved as KiCad 7 project
Parts:
- C1, C2: renamed from C?; value (none) -> 100n; footprint (none) -> Capacitor_SMD:C_0603_1608Metric
Changed lines of the file:
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@@
-(kicad_sch (version 20211123) (generator eeschema)
+(kicad_sch (version 20230121) (generator eeschema)
   (paper "A4")
   (title_block
@@
   )
   (wire (pts (xy 163.83 93.98) (xy 166.37 93.98))
-    (stroke (width 0) (type default) (color 0 0 0 0))
+    (stroke (width 0) (type default))
   )
   (wire (pts (xy 156.21 81.28) (xy 153.67 81.28))
-    (stroke (width 0) (type default) (color 0 0 0 0))
+    (stroke (width 0) (type default))
   )
   (wire (pts (xy 163.83 81.28) (xy 166.37 81.28))
-    (stroke (width 0) (type default) (color 0 0 0 0))
+    (stroke (width 0) (type default))
   )
   (wire (pts (xy 156.21 93.98) (xy 153.67 93.98))
-    (stroke (width 0) (type default) (color 0 0 0 0))
+    (stroke (width 0) (type default))
   )
-  (hierarchical_label "OUT-" (shape output) (at 153.67 93.98 180)
+  (hierarchical_label "OUT-" (shape output) (at 153.67 93.98 180) (fields_autoplaced)
     (effects (font (size 1.27 1.27)) (justify right))
   )
-  (hierarchical_label "IN-" (shape input) (at 166.37 93.98 0)
+  (hierarchical_label "IN-" (shape input) (at 166.37 93.98 0) (fields_autoplaced)
     (effects (font (size 1.27 1.27)) (justify left))
   )
-  (hierarchical_label "OUT+" (shape output) (at 153.67 81.28 180)
+  (hierarchical_label "OUT+" (shape output) (at 153.67 81.28 180) (fields_autoplaced)
     (effects (font (size 1.27 1.27)) (justify right))
   )
-  (hierarchical_label "IN+" (shape input) (at 166.37 81.28 0)
+  (hierarchical_label "IN+" (shape input) (at 166.37 81.28 0) (fields_autoplaced)
     (effects (font (size 1.27 1.27)) (justify left))
   )
   (symbol (lib_id "Device:C") (at 160.02 81.28 270) (unit 1)
-    (in_bom yes) (on_board yes)
-    (property "Reference" "C?" (id 0) (at 160.02 74.8792 90))
-    (property "Value" "" (id 1) (at 160.02 77.1906 90))
-    (property "Footprint" "" (id 2) (at 156.21 82.2452 0)
+    (in_bom yes) (on_board yes) (dnp no)
+    (property "Reference" "C1" (at 160.02 74.8792 90)
+      (effects (font (size 1.27 1.27)))
+    )
+    (property "Value" "100n" (at 160.02 77.1906 90)
+      (effects (font (size 1.27 1.27)))
+    )
+    (property "Footprint" "Capacitor_SMD:C_0603_1608Metric" (at 156.21 82.2452 0)
       (effects (font (size 1.27 1.27)) hide)
     )
-    (property "Datasheet" "~" (id 3) (at 160.02 81.28 0)
+    (property "Datasheet" "~" (at 160.02 81.28 0)
       (effects (font (size 1.27 1.27)) hide)
     )
     (pin "1")
     (pin "2")
+    (instances
+      (project "PCIexpress_x1_low"
+        (path "/b58173cd-28d5-49a4-a789-299fbf6f5cc2/00000000-0000-0000-0000-00005d508b15/00000000-0000-0000-0000-00005dab5272"
+          (reference "C1") (unit 1)
+        )
+      )
+    )
   )
   (symbol (lib_id "Device:C") (at 160.02 93.98 90) (mirror x) (unit 1)
-    (in_bom yes) (on_board yes)
-    (property "Reference" "C?" (id 0) (at 160.02 87.5792 90))
-    (property "Value" "" (id 1) (at 160.02 89.8906 90))
-    (property "Footprint" "" (id 2) (at 163.83 94.9452 0)
+    (in_bom yes) (on_board yes) (dnp no)
+    (property "Reference" "C2" (at 160.02 87.5792 90)
+      (effects (font (size 1.27 1.27)))
+    )
+    (property "Value" "100n" (at 160.02 89.8906 90)
+      (effects (font (size 1.27 1.27)))
+    )
+    (property "Footprint" "Capacitor_SMD:C_0603_1608Metric" (at 163.83 94.9452 0)
       (effects (font (size 1.27 1.27)) hide)
     )
-    (property "Datasheet" "~" (id 3) (at 160.02 93.98 0)
+    (property "Datasheet" "~" (at 160.02 93.98 0)
       (effects (font (size 1.27 1.27)) hide)
     )
     (pin "1")
     (pin "2")
+    (instances
+      (project "PCIexpress_x1_low"
+        (path "/b58173cd-28d5-49a4-a789-299fbf6f5cc2/00000000-0000-0000-0000-00005d508b15/00000000-0000-0000-0000-00005dab5272"
+          (reference "C2") (unit 1)
+        )
+      )
+    )
   )
 )
