File: PCIexpress_x1_low/term.kicad_sch (KiCad schematic)
At the start: 2 parts

Commit message: saved as KiCad 7 project
Parts:
- R1, R2: value (none) -> 49.9; footprint (none) -> Resistor_SMD:R_0603_1608Metric
Changed lines of the file:
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@@
-(kicad_sch (version 20211123) (generator eeschema)
+(kicad_sch (version 20230121) (generator eeschema)
   (paper "A4")
   (title_block
@@
   )
   (wire (pts (xy 146.05 90.17) (xy 148.59 90.17))
-    (stroke (width 0) (type default) (color 0 0 0 0))
+    (stroke (width 0) (type default))
   )
   (wire (pts (xy 146.05 92.71) (xy 146.05 90.17))
-    (stroke (width 0) (type default) (color 0 0 0 0))
+    (stroke (width 0) (type default))
   )
   (wire (pts (xy 143.51 90.17) (xy 146.05 90.17))
-    (stroke (width 0) (type default) (color 0 0 0 0))
+    (stroke (width 0) (type default))
   )
   (wire (pts (xy 120.65 92.71) (xy 120.65 90.17))
-    (stroke (width 0) (type default) (color 0 0 0 0))
+    (stroke (width 0) (type default))
   )
   (wire (pts (xy 146.05 100.33) (xy 146.05 102.87))
-    (stroke (width 0) (type default) (color 0 0 0 0))
+    (stroke (width 0) (type default))
   )
   (wire (pts (xy 120.65 90.17) (xy 123.19 90.17))
-    (stroke (width 0) (type default) (color 0 0 0 0))
+    (stroke (width 0) (type default))
   )
   (wire (pts (xy 118.11 90.17) (xy 120.65 90.17))
-    (stroke (width 0) (type default) (color 0 0 0 0))
+    (stroke (width 0) (type default))
   )
   (wire (pts (xy 120.65 100.33) (xy 120.65 102.87))
-    (stroke (width 0) (type default) (color 0 0 0 0))
+    (stroke (width 0) (type default))
   )
-  (hierarchical_label "IN-" (shape input) (at 123.19 90.17 0)
+  (hierarchical_label "IN-" (shape input) (at 123.19 90.17 0) (fields_autoplaced)
     (effects (font (size 1.27 1.27)) (justify left))
   )
-  (hierarchical_label "OUT+" (shape output) (at 143.51 90.17 180)
+  (hierarchical_label "OUT+" (shape output) (at 143.51 90.17 180) (fields_autoplaced)
     (effects (font (size 1.27 1.27)) (justify right))
   )
-  (hierarchical_label "IN+" (shape input) (at 148.59 90.17 0)
+  (hierarchical_label "IN+" (shape input) (at 148.59 90.17 0) (fields_autoplaced)
     (effects (font (size 1.27 1.27)) (justify left))
   )
-  (hierarchical_label "OUT-" (shape output) (at 118.11 90.17 180)
+  (hierarchical_label "OUT-" (shape output) (at 118.11 90.17 180) (fields_autoplaced)
     (effects (font (size 1.27 1.27)) (justify right))
   )
   (symbol (lib_id "Device:R") (at 120.65 96.52 0) (unit 1)
-    (in_bom yes) (on_board yes)
-    (property "Reference" "R1" (id 0) (at 122.428 95.3516 0)
+    (in_bom yes) (on_board yes) (dnp no)
+    (property "Reference" "R1" (at 122.428 95.3516 0)
       (effects (font (size 1.27 1.27)) (justify left))
     )
-    (property "Value" "" (id 1) (at 122.428 97.663 0)
+    (property "Value" "49.9" (at 122.428 97.663 0)
       (effects (font (size 1.27 1.27)) (justify left))
     )
-    (property "Footprint" "" (id 2) (at 118.872 96.52 90)
+    (property "Footprint" "Resistor_SMD:R_0603_1608Metric" (at 118.872 96.52 90)
       (effects (font (size 1.27 1.27)) hide)
     )
-    (property "Datasheet" "~" (id 3) (at 120.65 96.52 0)
+    (property "Datasheet" "~" (at 120.65 96.52 0)
       (effects (font (size 1.27 1.27)) hide)
     )
     (pin "1")
     (pin "2")
+    (instances
+      (project "PCIexpress_x1_low"
+        (path "/b58173cd-28d5-49a4-a789-299fbf6f5cc2/00000000-0000-0000-0000-00005d508b15/00000000-0000-0000-0000-00005d516dfb"
+          (reference "R1") (unit 1)
+        )
+      )
+    )
   )
   (symbol (lib_id "Device:R") (at 146.05 96.52 0) (unit 1)
-    (in_bom yes) (on_board yes)
-    (property "Reference" "R2" (id 0) (at 147.828 95.3516 0)
+    (in_bom yes) (on_board yes) (dnp no)
+    (property "Reference" "R2" (at 147.828 95.3516 0)
       (effects (font (size 1.27 1.27)) (justify left))
     )
-    (property "Value" "" (id 1) (at 147.828 97.663 0)
+    (property "Value" "49.9" (at 147.828 97.663 0)
       (effects (font (size 1.27 1.27)) (justify left))
     )
-    (property "Footprint" "" (id 2) (at 144.272 96.52 90)
+    (property "Footprint" "Resistor_SMD:R_0603_1608Metric" (at 144.272 96.52 90)
       (effects (font (size 1.27 1.27)) hide)
     )
-    (property "Datasheet" "~" (id 3) (at 146.05 96.52 0)
+    (property "Datasheet" "~" (at 146.05 96.52 0)
       (effects (font (size 1.27 1.27)) hide)
     )
     (pin "1")
     (pin "2")
+    (instances
+      (project "PCIexpress_x1_low"
+        (path "/b58173cd-28d5-49a4-a789-299fbf6f5cc2/00000000-0000-0000-0000-00005d508b15/00000000-0000-0000-0000-00005d516dfb"
+          (reference "R2") (unit 1)
+        )
+      )
+    )
   )
   (symbol (lib_id "power:GND") (at 120.65 102.87 0) (unit 1)
-    (in_bom yes) (on_board yes)
-    (property "Reference" "#PWR0109" (id 0) (at 120.65 109.22 0)
+    (in_bom yes) (on_board yes) (dnp no)
+    (property "Reference" "#PWR0109" (at 120.65 109.22 0)
       (effects (font (size 1.27 1.27)) hide)
     )
-    (property "Value" "" (id 1) (at 120.777 107.2642 0))
-    (property "Footprint" "" (id 2) (at 120.65 102.87 0)
+    (property "Value" "GND" (at 120.777 107.2642 0)
+      (effects (font (size 1.27 1.27)))
+    )
+    (property "Footprint" "" (at 120.65 102.87 0)
       (effects (font (size 1.27 1.27)) hide)
     )
-    (property "Datasheet" "" (id 3) (at 120.65 102.87 0)
+    (property "Datasheet" "" (at 120.65 102.87 0)
       (effects (font (size 1.27 1.27)) hide)
     )
     (pin "1")
+    (instances
+      (project "PCIexpress_x1_low"
+        (path "/b58173cd-28d5-49a4-a789-299fbf6f5cc2/00000000-0000-0000-0000-00005d508b15/00000000-0000-0000-0000-00005d516dfb"
+          (reference "#PWR0109") (unit 1)
+        )
+      )
+    )
   )
   (symbol (lib_id "power:GND") (at 146.05 102.87 0) (unit 1)
-    (in_bom yes) (on_board yes)
-    (property "Reference" "#PWR0110" (id 0) (at 146.05 109.22 0)
+    (in_bom yes) (on_board yes) (dnp no)
+    (property "Reference" "#PWR0110" (at 146.05 109.22 0)
       (effects (font (size 1.27 1.27)) hide)
     )
-    (property "Value" "" (id 1) (at 146.177 107.2642 0))
-    (property "Footprint" "" (id 2) (at 146.05 102.87 0)
+    (property "Value" "GND" (at 146.177 107.2642 0)
+      (effects (font (size 1.27 1.27)))
+    )
+    (property "Footprint" "" (at 146.05 102.87 0)
       (effects (font (size 1.27 1.27)) hide)
     )
-    (property "Datasheet" "" (id 3) (at 146.05 102.87 0)
+    (property "Datasheet" "" (at 146.05 102.87 0)
       (effects (font (size 1.27 1.27)) hide)
     )
     (pin "1")
+    (instances
+      (project "PCIexpress_x1_low"
+        (path "/b58173cd-28d5-49a4-a789-299fbf6f5cc2/00000000-0000-0000-0000-00005d508b15/00000000-0000-0000-0000-00005d516dfb"
+          (reference "#PWR0110") (unit 1)
+        )
+      )
+    )
   )
 )
